File: PCB/FT232H-ATF150x.kicad_sch (KiCad schematic)
At the start: 18 parts, among them J1 CJMCU-232H, J2 JTAG-Altera, U1 ATF150x-xJx44, U2 MAX662A

Commit message: comments & silkscreen
Parts:
- J2: value JTAG-Altera -> Altera JTAG-A+VPP; symbol 000_LOCAL:JTAG-Altera -> 000_LOCAL:Altera JTAG-A+VPP
- U1: value ATF150x-xJx44 -> ATF150x-xJx44 (PLCC-44); symbol 000_LOCAL:ATF150x-xJx44 -> 000_LOCAL:ATF150x-xJx44 (PLCC-44)
Connections:
- net +12V: now also R1.2; no longer R1.1
- net at JP2.2 (C): now also R1.1; no longer R1.2
- net OE1 renamed VPP
Other:
- note added: "(1)"
- note added: "(1) VPP on JTAG pin 6 is a non-standard extension. It should be ignored by most targets as pin 6 is usually nc, and also only applies when JP2 is shorted."
- moved on the sheet: C1, C2, C3, C4, JP2, R1
