File: PCB/ATF150x_uPRG_sw.kicad_pcb (KiCad board)
At the start: 2 copper layers, 38.1 x 22.9 mm, 29 parts, among them J1 Adafruit_2264, J2 Altera JTAG-A+VPP, SW1 SP3T, SW2 SPDT, U1 MAX662A

Commit message: _sw fillet tracks
Routing:
- net +5V: track 29.8 -> 31.3 mm
- net Net-(SW2-B): track 17.6 -> 17.1 mm
